Commit message: Added object detection and color identification code

File: simulation/models/box.urdf (robot description, URDF)
Before this commit: robot aruco, 1 links, 0 joints
Links:
- link simple_box_base_link: geometry collision box size=1.0 1.0 0.4; visual mesh filename=/home/deep/catkin_ws/src/simulation/models/meshes/box.dae
